Commit message: Add actual masses to 3D model.

File: models/CatModel.urdf (robot description, URDF)
Before this commit: robot CatModel, 33 links, 32 joints
Links:
- link Battery1: mass 0.6539897585243583 -> 0.41
- link Electronics1: mass 0.1587634595739255 -> 0.24
- link Head1: mass 0.8146696853490065 -> 0.15
- link Head_Servo1: mass 0.07800761310887962 -> 0.13
- link Left_Front_Joint1: mass 0.0049939542219629126 -> 0.000001
- link Left_Front_Paw1: mass 0.009860673647584237 -> 0.000001
- link Left_Rear_Joint1: mass 0.0049939542219629126 -> 0.000001
- link Left_Rear_Paw1: mass 0.009860673647584237 -> 0.000001
- link Lower_Left_Front_Leg1: mass 0.012527915218877713 -> 0.045
- link Lower_Left_Front_Servo1: mass 0.08509975852435851 -> 0.13
- link Lower_Left_Rear_Leg1: mass 0.012527915218877675 -> 0.045
- link Lower_Left_Rear_Servo1: mass 0.0850997585243585 -> 0.13
- link Lower_Right_Front_Leg1: mass 0.012527915218877713 -> 0.045
- link Lower_Right_Front_Servo1: mass 0.0850997585243585 -> 0.13
- link Lower_Right_Rear_Leg1: mass 0.012527915218877675 -> 0.045
- link Lower_Right_Rear_Servo1: mass 0.08509975852435848 -> 0.13
- link Neck1: mass 0.19671474883465964 -> 0.05
- link Neck_Servo1: mass 0.08701463778653835 -> 0.13
- link Right_Front_Joint1: mass 0.0049939542219628675 -> 0.000001
- link Right_Front_Paw1: mass 0.009860673647584237 -> 0.000001
- link Right_Rear_Joint1: mass 0.0049939542219628675 -> 0.000001
- link Right_Rear_Paw1: mass 0.009860673647584237 -> 0.000001
- link Tail1: mass 0.01723009674422482 -> 0.05
- link Tail_Servo1: mass 0.08689583836578228 -> 0.13
- link Upper_Left_Front_Leg1: mass 0.014216059949049762 -> 0.045
- link Upper_Left_Front_Servo1: mass 0.08892951704871721 -> 0.13
- link Upper_Left_Rear_Leg1: mass 0.014216059949049762 -> 0.045
- link Upper_Left_Rear_Servo1: mass 0.08892951704871722 -> 0.13
- link Upper_Right_Front_Leg1: mass 0.014216059949049762 -> 0.045
- link Upper_Right_Front_Servo1: mass 0.08892951704871722 -> 0.13
- link Upper_Right_Rear_Leg1: mass 0.014216059949049762 -> 0.045
- link Upper_Right_Rear_Servo1: mass 0.08892951704871728 -> 0.13
- link base_link: mass 0.23060219033668225 -> 0.37
